File: hardware/ESP32DevKitCv4_SA8x8_Ver_B.brd (EAGLE design)
At the start: 82.7 x 61.6 mm, 56 parts, among them J1 POWER_JACKPTH_LOCK, J2 XT60PW-M, T1 2N3904

Commit message: WIP: HW VerB in progress
Parts:
- added C19, C20: 100n, resistor:C0805
- added R22: 10k, resistor:R0805
- added R23, R24: 1k, resistor:R0805
- moved R21 106.8 mm to (47.6, 56.5), flipped to the bottom, turned to 270 degrees
- moved R20 98.9 mm to (42.5, 56.5), flipped to the bottom, turned to 90 degrees
- moved C17 63.0 mm to (6.83, 44.5), turned to 180 degrees
- moved C18 62.0 mm to (6.83, 37.3), turned to 180 degrees
- moved C16 52.4 mm to (6.83, 39.8)
Connections:
- net SCL renamed OLED_SCL
- net SDA renamed OLED_SDA
- new net ROT_CLK_ROUTE: R21.1, R24.1, S1.A
- new net ROT_DAT_ROUTE: R20.2, R23.1, S1.B
- net +3V3: now also C20.2, R20.1, R21.2, R22.1
- net +5V: now also C19.2
- net GND: now also C19.1, C20.1; no longer R20.1, R21.2
- net ROT_BTN: now also R22.2
- net ROT_CLK: now also R24.2; no longer R21.1, S1.A
- net ROT_DAT: now also R23.2; no longer R20.2, S1.B
Routing:
- net ROT_CLK: track 61.3 -> 5.79 mm
- net ROT_CLK_ROUTE: track 0.00 -> 52.8 mm
- net ROT_DAT: track 51.1 -> 6.85 mm
- net ROT_DAT_ROUTE: track 0.00 -> 42.4 mm
- net +3V3: track 58.5 -> 90.4 mm, vias 2 -> 4
- net +5V: track 139.2 -> 129.1 mm, vias 7 -> 5
- net N$14: track 21.1 -> 23.4 mm
- net GND: track 0.17 -> 1.80 mm, vias 40 -> 63
- net ROT_BTN: track 52.6 -> 54.1 mm
Other:
- board text added: "APRS-ESP32 V1.5B"
- board text added: "github.com/erstec/APRS-ESP"
- board text removed: "ESP32-DevKitC-v4 SA8x8 V1.5B"
- board text removed: "github.com/erstec/ESP32IGate"

Commit message: WIP: pinout Corrections after tests
Connections:
- net POW: now also U$1.9; no longer U$1.13
Routing:
- net POW: track 50.8 -> 64.0 mm
Changed lines of the file:
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@@
 <contactref element="DRA818V" pad="7"/>
 <contactref element="C8" pad="1"/>
-<wire x1="69.965" y1="31.3575" x2="69.965" y2="31.4325" width="0.4064" layer="1"/>
-<wire x1="69.965" y1="31.4325" x2="69.965" y2="34.8125" width="0.4064" layer="1"/>
+<wire x1="69.965" y1="31.3575" x2="69.965" y2="34.8125" width="0.4064" layer="1"/>
 <wire x1="69.965" y1="34.8125" x2="69.85" y2="34.9275" width="0.4064" layer="1"/>
-<contactref element="U$1" pad="13"/>
 <wire x1="61.4675" y1="26.3525" x2="64.0075" y2="28.8925" width="0.4064" layer="1"/>
 <wire x1="38.67785" y1="27.56030625" x2="38.67785" y2="29.21" width="0.4064" layer="1"/>
 <wire x1="38.67785" y1="29.21" x2="38.57625" y2="29.3116" width="0.4064" layer="1"/>
 <wire x1="38.57625" y1="29.3116" x2="31.17215" y2="29.3116" width="0.4064" layer="1"/>
-<wire x1="31.115" y1="29.36875" x2="31.17215" y2="29.3116" width="0.4064" layer="1"/>
-<via x="31.115" y="29.36875" extent="1-16" drill="0.35" shape="octagon"/>
 <wire x1="61.4675" y1="26.3525" x2="39.88565625" y2="26.3525" width="0.4064" layer="1"/>
 <wire x1="39.88565625" y1="26.3525" x2="38.67785" y2="27.56030625" width="0.4064" layer="1"/>
-<wire x1="31.115" y1="29.36875" x2="31.115" y2="28.09875" width="0.4064" layer="16"/>
-<via x="31.115" y="28.09875" extent="1-16" drill="0.35" shape="octagon"/>
-<wire x1="31.115" y1="28.09875" x2="28.86075" y2="28.09875" width="0.4064" layer="1"/>
-<wire x1="28.86075" y1="28.09875" x2="28.692" y2="28.2675" width="0.4064" layer="1"/>
 <wire x1="64.0075" y1="28.8925" x2="67.945" y2="28.8925" width="0.4064" layer="1"/>
 <wire x1="67.945" y1="28.8925" x2="69.965" y2="30.9125" width="0.4064" layer="1"/>
 <wire x1="69.965" y1="30.9125" x2="69.965" y2="31.3575" width="0.4064" layer="1"/>
+<contactref element="U$1" pad="9"/>
+<via x="31.17215" y="29.3116" extent="1-16" drill="0.35" shape="octagon"/>
+<wire x1="31.17215" y1="29.3116" x2="30.95625" y2="29.0957" width="0.4064" layer="16"/>
+<wire x1="30.95625" y1="29.0957" x2="30.95625" y2="27.94" width="0.4064" layer="16"/>
+<via x="30.95625" y="27.94" extent="1-16" drill="0.35" shape="octagon"/>
+<wire x1="30.95625" y1="27.94" x2="30.196475" y2="27.94" width="0.4064" layer="1"/>
+<wire x1="30.196475" y1="27.94" x2="29.253975" y2="26.9975" width="0.4064" layer="1"/>
+<wire x1="29.253975" y1="26.9975" x2="29.243975" y2="26.9875" width="0.3048" layer="1"/>
+<wire x1="29.243975" y1="26.9875" x2="28.09875" y2="26.9875" width="0.3048" layer="1"/>
+<wire x1="28.09875" y1="26.9875" x2="27.305" y2="27.78125" width="0.4064" layer="1"/>
+<wire x1="27.305" y1="37.0405" x2="28.692" y2="38.4275" width="0.4064" layer="1"/>
+<wire x1="27.305" y1="27.78125" x2="27.305" y2="37.0405" width="0.4064" layer="1"/>
 </signal>
 <signal name="PD">
