File: hardware/ESP32DevKitCv4_SA8x8_Ver_B.sch (EAGLE design)
At the start: 56 parts, among them J1 POWER_JACKPTH_LOCK, J2 XT60PW-M, T1 2N3904

Commit message: WIP: HW VerB in progress
Parts:
- added C19, C20: 100n, resistor:C-EUC0805
- added R22: 10k, resistor:R-US_R0805
- added R23, R24: 1k, resistor:R-US_R0805
Connections:
- net SCL renamed OLED_SCL
- net SDA renamed OLED_SDA
- new net ROT_CLK_ROUTE: R21.1, R24.1, S1.A
- new net ROT_DAT_ROUTE: R20.2, R23.1, S1.B
- net +3V3: now also C20.2, R20.1, R21.2, R22.1
- net +5V: now also C19.2
- net GND: now also C19.1, C20.1; no longer R20.1, R21.2
- net ROT_BTN: now also R22.2
- net ROT_CLK: now also R24.2; no longer R21.1, S1.A
- net ROT_DAT: now also R23.2; no longer R20.2, S1.B
Other:
- note added: "LY3PH"
- note removed: "Redesigned by LY3PH"
- moved on the sheet: C16, C17, R20, R21

Commit message: WIP: pinout Corrections after tests
Connections:
- net POW: now also U$1.IO25; no longer U$1.IO12
Changed lines of the file:
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@@
 </segment>
 <segment>
-<pinref part="U$1" gate="G$1" pin="IO12"/>
-<wire x1="27.94" y1="88.9" x2="20.32" y2="88.9" width="0.1524" layer="91"/>
-<label x="20.32" y="88.9" size="1.778" layer="95"/>
+<wire x1="27.94" y1="99.06" x2="20.32" y2="99.06" width="0.1524" layer="91"/>
+<pinref part="U$1" gate="G$1" pin="IO25"/>
+<label x="20.32" y="99.06" size="1.778" layer="95"/>
 </segment>
 </net>
