File: hardware/ESP32DevKitCv4_SA8x8_Rev_B.brd (EAGLE design)
At the start: 82.7 x 61.6 mm, 56 parts, among them J1 POWER_JACKPTH_LOCK, J2 XT60PW-M, T1 2N3904

Commit message: DONE: Rev.B
Parts:
- added C19, C20: 100n, resistor:C0805
- added R22: 10k, resistor:R0805
- added R23, R24: 1k, resistor:R0805
- moved R21 106.8 mm to (47.6, 56.5), flipped to the bottom, turned to 270 degrees
- moved R20 98.9 mm to (42.5, 56.5), flipped to the bottom, turned to 90 degrees
- moved C17 63.0 mm to (6.83, 44.5), turned to 180 degrees
- moved C18 62.0 mm to (6.83, 37.3), turned to 180 degrees
- moved C16 52.4 mm to (6.83, 39.8)
Connections:
- net SCL renamed OLED_SCL
- net SDA renamed OLED_SDA
- new net ROT_CLK_ROUTE: R21.1, R24.1, S1.A
- new net ROT_DAT_ROUTE: R20.2, R23.1, S1.B
- net +3V3: now also C20.2, R20.1, R21.2, R22.1
- net +5V: now also C19.2
- net GND: now also C19.1, C20.1; no longer R20.1, R21.2
- net POW: now also U$1.9; no longer U$1.13
- net ROT_BTN: now also R22.2
- net ROT_CLK: now also R24.2; no longer R21.1, S1.A
- net ROT_DAT: now also R23.2; no longer R20.2, S1.B
Routing:
- net ROT_CLK: track 61.3 -> 5.79 mm
- net ROT_CLK_ROUTE: track 0.00 -> 52.8 mm
- net ROT_DAT: track 51.1 -> 6.85 mm
- net ROT_DAT_ROUTE: track 0.00 -> 42.4 mm
- net +3V3: track 58.5 -> 90.4 mm, vias 2 -> 4
- net POW: track 50.5 -> 64.0 mm
- net +5V: track 139.2 -> 129.1 mm, vias 7 -> 5
- net N$14: track 21.1 -> 23.4 mm
- net GND: track 0.17 -> 1.80 mm, vias 40 -> 347
- net ROT_BTN: track 52.6 -> 54.1 mm
Other:
- board text added: "APRS-ESP32 V1.5 Rev.B"
- board text added: "github.com/erstec/APRS-ESP"
- board text removed: "ESP32-DevKitC-v4 SA8x8 V1.5B"
- board text removed: "github.com/erstec/ESP32IGate"
