File: hardware/APRS-ESP32_SA8x8_Rev_B.brd (EAGLE design)
At the start: 82.7 x 61.6 mm, 61 parts, among them J1 POWER_JACKPTH_LOCK, J2 XT60PW-M, T1 2N3904

Commit message: WIP: Rev.C
Connections:
- net RXD_DRJ renamed RXD_RF
- net TXD_DRJ renamed TXD_RF
Changed lines of the file:
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@@
 <wire x1="29.2" y1="35.8875" x2="28.692" y2="35.8875" width="0.4064" layer="16"/>
-</signal>
-<signal name="TXD_DRJ">
-<contactref element="U$1" pad="12"/>
-<contactref element="R12" pad="2"/>
-<wire x1="30.82925" y1="28.702" x2="30.48" y2="29.05125" width="0.4064" layer="1"/>
-<wire x1="30.48" y1="29.05125" x2="30.48" y2="29.68625" width="0.4064" layer="1"/>
-<wire x1="30.48" y1="29.68625" x2="29.36875" y2="30.7975" width="0.4064" layer="1"/>
-<wire x1="29.36875" y1="30.7975" x2="29.327" y2="30.8075" width="0.4064" layer="1"/>
-<wire x1="29.327" y1="30.8075" x2="28.692" y2="30.8075" width="0.4064" layer="1"/>
-<wire x1="33.02" y1="25.08" x2="31.75" y2="26.35" width="0.4064" layer="1"/>
-<wire x1="31.75" y1="28.30195625" x2="31.34995625" y2="28.702" width="0.4064" layer="1"/>
-<wire x1="31.75" y1="26.35" x2="31.75" y2="28.30195625" width="0.4064" layer="1"/>
-<wire x1="31.34995625" y1="28.702" x2="30.82925" y2="28.702" width="0.4064" layer="1"/>
-</signal>
-<signal name="RXD_DRJ">
-<contactref element="U$1" pad="15"/>
-<contactref element="R11" pad="2"/>
-<wire x1="28.692" y1="23.1875" x2="28.72375" y2="23.1875" width="0.4064" layer="1"/>
-<wire x1="31.1175" y1="20.79375" x2="33.02" y2="20.79375" width="0.4064" layer="1"/>
-<wire x1="28.72375" y1="23.1875" x2="31.1175" y2="20.79375" width="0.4064" layer="1"/>
 </signal>
 <signal name="POW">
@@
 <wire x1="27.94" y1="47.3075" x2="27.14625" y2="48.10125" width="0.4064" layer="1"/>
 </signal>
+<signal name="RXD_RF">
+<contactref element="R11" pad="2"/>
+<contactref element="U$1" pad="15"/>
+<wire x1="28.692" y1="23.1875" x2="28.72375" y2="23.1875" width="0.4064" layer="1"/>
+<wire x1="28.72375" y1="23.1875" x2="31.1175" y2="20.79375" width="0.4064" layer="1"/>
+<wire x1="31.1175" y1="20.79375" x2="33.02" y2="20.79375" width="0.4064" layer="1"/>
+</signal>
+<signal name="TXD_RF">
+<contactref element="R12" pad="2"/>
+<contactref element="U$1" pad="12"/>
+<wire x1="30.82925" y1="28.702" x2="30.48" y2="29.05125" width="0.4064" layer="1"/>
+<wire x1="30.48" y1="29.05125" x2="30.48" y2="29.68625" width="0.4064" layer="1"/>
+<wire x1="30.48" y1="29.68625" x2="29.36875" y2="30.7975" width="0.4064" layer="1"/>
+<wire x1="29.36875" y1="30.7975" x2="29.327" y2="30.8075" width="0.4064" layer="1"/>
+<wire x1="29.327" y1="30.8075" x2="28.692" y2="30.8075" width="0.4064" layer="1"/>
+<wire x1="31.75" y1="28.30195625" x2="31.34995625" y2="28.702" width="0.4064" layer="1"/>
+<wire x1="31.75" y1="28.30195625" x2="31.75" y2="26.35" width="0.4064" layer="1"/>
+<wire x1="31.34995625" y1="28.702" x2="30.82925" y2="28.702" width="0.4064" layer="1"/>
+<wire x1="31.75" y1="26.35" x2="33.02" y2="25.08" width="0.4064" layer="1"/>
+</signal>
 </signals>
