File: hardware/APRS-ESP32_SA8x8_Rev_B.sch (EAGLE design)
At the start: 61 parts, among them J1 POWER_JACKPTH_LOCK, J2 XT60PW-M, T1 2N3904

Commit message: WIP: Rev.C
Connections:
- net RXD_DRJ renamed RXD_RF
- net TXD_DRJ renamed TXD_RF
Other:
- moved on the sheet: ANT1, ANT2, C1, C11, C12, C13, C14, C15, C16, C17, C18, C19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
