File: hardware/APRS-ESP32_SA8x8_Rev_C.brd (EAGLE design)
At the start: 82.7 x 61.6 mm, 71 parts, among them IC2 LD117AS12TR, J1 POWER_JACKPTH_LOCK, J2 XT60PW-M, T1 2N3904

Commit message: WIP: Rev.C
Parts:
- added C24: 100n, resistor:C0805
- added R27, R28: 10k, resistor:R0805
- UART1: value GND TX RX + -> + R B T R G; device pinhead:1X04 -> con-lstb:MA06-1
- moved UART1 55.1 mm to (-6.35, -48.9)
- moved U$2 54.1 mm to (25.9, 14.3), turned to 90 degrees
- moved J1 22.9 mm to (76.8, 61.6)
- moved J2 3.18 mm to (64.3, 51.1)
Connections:
- removed net IN-: J2.2
- removed net ROT_BTN: C18.2, R22.2, S1.SW+, U$2.IO5
- new net BOOT/ROT_BTN: C18.2, R22.2, R28.2, S1.SW+, U$2.IO0, U$2.IO5, UART1.4
- new net RST: C24.2, R27.2, U$2.EN, UART1.5
- net +3V3: now also R27.1, R28.1, UART1.6
- net +5V: no longer UART1.1
- net GND: now also C24.1, J2.2, U$2.GND2, U$2.GND3, UART1.1; no longer UART1.4
Routing:
- net +3V3: track 58.5 -> 27.5 mm
- net AF_IN: track 37.4 -> 18.7 mm, vias 1 -> 0
- net ROT_BTN: track 2.32 -> 0.00 mm
- net BOOT/ROT_BTN: track 0.00 -> 2.32 mm
Other:
- outline, holes or cut-outs redrawn
