File: hardware/APRS-ESP32_SA8x8_Rev_C.sch (EAGLE design)
At the start: 71 parts, among them IC2 LD117AS12TR, J1 POWER_JACKPTH_LOCK, J2 XT60PW-M, T1 2N3904

Commit message: WIP: Rev.C
Parts:
- added C24: 100n, resistor:C-EUC0805
- added R27, R28: 10k, resistor:R-US_R0805
- UART1: value GND TX RX + -> + R B T R G; device pinhead:PINHD-1X4 -> con-lstb:MA06-1
Connections:
- removed net IN-: J2.-
- removed net ROT_BTN: C18.2, R22.2, S1.SW+, U$2.GPIO5
- new net BOOT/ROT_BTN: C18.2, R22.2, R28.2, S1.SW+, U$2.GPIO0, U$2.GPIO5, UART1.4
- new net RST: C24.2, R27.2, U$2.EN, UART1.5
- net +3V3: now also R27.1, R28.1, UART1.6
- net +5V: no longer UART1.1
- net GND: now also C24.1, J2.-, U$2.GND2, U$2.GND3, UART1.1; no longer UART1.4
Other:
- moved on the sheet: ANT1, ANT2, C1, C11, C12, C13, C14, C15, C16, C17, C18, C19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
