File: hardware/APRS-ESP32_SA8x8_Rev_D.sch (EAGLE design)
At the start: 61 parts, among them J1 POWER_JACKPTH_LOCK, J2 XT60PW-M, T1 2N3904

Commit message: Stable
R10 560 -> 680
R11, R12 100 -> 0
Gerbers added
Parts:
- R10: value 560 -> 680
- R11, R12: value 100 -> 0
Changed lines of the file:
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@@
 <part name="GND26" library="supply1" library_urn="urn:adsk.eagle:library:371" deviceset="GND" device=""/>
 <part name="GND19" library="supply1" library_urn="urn:adsk.eagle:library:371" deviceset="GND" device=""/>
-<part name="R10" library="resistor" deviceset="R-US_" device="R0805" value="560"/>
-<part name="R11" library="resistor" deviceset="R-US_" device="R0805" value="100"/>
-<part name="R12" library="resistor" deviceset="R-US_" device="R0805" value="100"/>
+<part name="R10" library="resistor" deviceset="R-US_" device="R0805" value="680"/>
+<part name="R11" library="resistor" deviceset="R-US_" device="R0805" value="0"/>
+<part name="R12" library="resistor" deviceset="R-US_" device="R0805" value="0"/>
 <part name="R13" library="resistor" deviceset="R-US_" device="R0805" value="100"/>
 <part name="R14" library="resistor" deviceset="R-US_" device="R0805" value="100"/>
