File: hardware/audio-adapter.brd (EAGLE design)
At the start: 18.1 x 29.2 mm, 21 parts

Commit message: - T-TWR PLUS V2.0 MOD board support added
- ESP32S3 -> ESP32E adapter Rev.C added
- AudioAdapter BOM fix (4k7->33k)
- README.md updated
Parts:
- R8: value 4k7 -> 4k7 / 33k
Changed lines of the file:
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@@
 <attribute name="VALUE" x="13.335" y="19.05" size="1.27" layer="27"/>
 </element>
-<element name="R8" library="resistor" package="R0805" value="4k7" x="9.525" y="6.35" smashed="yes" rot="R270">
+<element name="R8" library="resistor" package="R0805" value="4k7 / 33k" x="9.525" y="6.35" smashed="yes" rot="R270">
 <attribute name="NAME" x="10.795" y="6.985" size="1.27" layer="25" rot="R270"/>
 <attribute name="VALUE" x="6.985" y="6.985" size="1.27" layer="27" rot="R270"/>
